Commit message: 4輪モデルの修正

File: ros2_ws/src/raspbot_description/urdf/raspbot.urdf.xacro (robot description, xacro)
@@ -46,5 +46,5 @@
       </inertial>
       <visual>
-        <origin xyz="0 0 0" rpy="0 1.57079632679 0"/>
+        <origin xyz="0 0 0" rpy="1.57079632679 0 0"/>
         <geometry>
           <cylinder radius="${wheel_radius}" length="${wheel_width}"/>
@@ -55,5 +55,5 @@
       </visual>
       <collision>
-        <origin xyz="0 0 0" rpy="0 1.57079632679 0"/>
+        <origin xyz="0 0 0" rpy="1.57079632679 0 0"/>
         <geometry>
           <cylinder radius="${wheel_radius}" length="${wheel_width}"/>
